File: hardware/novy/novy.kicad_sch (KiCad schematic)
At the start: 36 parts, among them J1 RJ45, J2 SAFETY_SW, SW1 SW_Rotary_1x12, SW2 SW_Rotary_1x12, SW3 SW_Rotary_1x12, U1 Beetle ESP32-C6, U2 MCP2562-E-P, U3 PCA9685PW

Commit message: working prototype
Parts:
- added R13: 120, Resistor_SMD:R_1206_3216Metric_Pad1.30x1.75mm_HandSolder, symbol Device:R
- C1, C2, C3, C4, C5: value C -> 100nF
- R1: footprint Resistor_SMD:R_0603_1608Metric_Pad0.98x0.95mm_HandSolder -> Resistor_SMD:R_1206_3216Metric_Pad1.30x1.75mm_HandSolder; now left out of the parts list
- R10, R11, R12, R2, R3, R4, R5, R6, R7, R8, R9: footprint Resistor_SMD:R_0603_1608Metric_Pad0.98x0.95mm_HandSolder -> Resistor_SMD:R_1206_3216Metric_Pad1.30x1.75mm_HandSolder
Connections:
- net +3.3V: now also J1.5
- net CANH: now also R13.1
- net CANL: now also R13.2
- net PAN_CLK: now reaches J1.6
- net PAN_CLK: now also U1.5 (GPIO23)
- removed net PRES: J1.5, U1.5 (GPIO23)
- no-connect marks 26 -> 25
Other:
- moved on the sheet: C6, R1, R2
