File: hardware/novy/novy.kicad_pcb (KiCad board)
At the start: 2 copper layers, 160 x 60 mm, 36 parts, among them J1 RJ45, J2 SAFETY_SW, SW1 SW_Rotary_1x12, SW2 SW_Rotary_1x12, SW3 SW_Rotary_1x12, U1 Beetle ESP32-C6, U2 MCP2562-E-P, U3 PCA9685PW

Commit message: working prototype
Parts:
- added R13: 120, Resistor_SMD:R_1206_3216Metric_Pad1.30x1.75mm_HandSolder, F.Cu at (184.8, 67.2)
- C1, C2, C3, C4, C5: value C -> 100nF
- R1, R10, R11, R12, R2, R3, R4, R5, R6, R7, R8, R9: footprint Resistor_SMD:R_0603_1608Metric_Pad0.98x0.95mm_HandSolder -> Resistor_SMD:R_1206_3216Metric_Pad1.30x1.75mm_HandSolder
- moved R3 2.11 mm to (77.5, 55.1)
- moved R7 2.08 mm to (77.5, 61.0)
- moved R2 1.72 mm to (155.2, 78.1)
- moved R1 0.70 mm to (149.3, 75.4)
- moved R12 0.65 mm to (155.2, 80.6)
- moved R4 0.50 mm to (152.2, 55.5)
- moved R5 0.49 mm to (165.8, 55.4)
- moved R11 0.46 mm to (183.9, 55.0)
- moved R6 0.40 mm to (152.2, 60.6)
- moved R8 0.29 mm to (165.9, 60.5), turned to -90 degrees
Connections:
- J1 pad 5: PRES -> +3.3V
- J1 pad 6: unconnected-(J1-Pad6) -> PAN_CLK
- U1 pad 5: PRES -> PAN_CLK
Routing:
- net PRES: track 51.0 -> 0.00 mm, vias 2 -> 0
- net PAN_CLK: track 0.00 -> 48.6 mm, vias 0 -> 2
- net +3.3V: track 260.3 -> 271.7 mm
- net Net-(U3-LED0): track 25.6 -> 28.5 mm
- net CANH: track 14.5 -> 17.2 mm
- net Net-(J2-Pin_3): track 74.8 -> 72.4 mm
- net INTA: track 101.1 -> 99.0 mm
- net SCK: track 115.9 -> 117.9 mm
- net Net-(PAN1-A): track 2.85 -> 4.83 mm
- net Net-(ST2-KA): track 5.63 -> 7.41 mm
- net Net-(U3-LED2): track 33.2 -> 34.9 mm
- net Net-(ST2-AK): track 123.5 -> 124.7 mm
- net Net-(U3-LED4): track 120.9 -> 120.0 mm
- net CANL: track 10.4 -> 11.2 mm
- net GND: track 24.8 -> 24.2 mm
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
Commit message: working firmware
Routing:
- net Net-(U1-GPIO17): track 115.6 -> 114.3 mm
- net +3.3V: track 271.7 -> 272.7 mm
- net Net-(IO_SW3-GPB1): track 32.8 -> 33.6 mm
- net Net-(IO_SW3-GPA0): track 30.5 -> 29.8 mm
- net Net-(IO_SW2-GPB1): track 31.2 -> 32.0 mm
- net GND: vias 4 -> 16
- added copper zone on F.Cu, net GND
